File: pcb/touch/card_lights.sch (KiCad schematic (older format))
At the start: 28 parts, among them J1 TOUCH PAD, J2 LED_PAD, J3 LED_PAD, J4 LED_PAD, J5 LED_WIRE, J6 LED_WIRE, J7 LED_WIRE, U1 ATtiny10-TS, U2 TTP223E-HA6

Commit message: add new components, start making pretty for PCB manufacture
Parts:
- removed D7: D, Diode_SMD:D_SOD-123F, symbol Device:D
- added JP1: PROG, Jumper:SolderJumper-2_P1.3mm_Bridged_RoundedPad1.0x1.5mm, symbol Device:Jumper_NC_Small
Connections:
- net PB3: now also JP1.1
- net at U2.1 (Q): now also JP1.2
Other:
- note added: "Cut jumper before programming"
Changed lines of the file:
@@
 Text Notes 8850 2450 0    50   ~ 0
 For touch pad use flood fill on PCB back
-$Comp
-L Device:D D7
-U 1 1 5FF0713E
-P 5250 2400
-F 0 "D7" H 5250 2500 50  0000 C CNN
-F 1 "D" H 5250 2300 50  0000 C CNN
-F 2 "Diode_SMD:D_SOD-123F" H 5250 2400 50  0001 C CNN
-F 3 "~" H 5250 2400 50  0001 C CNN
-	1    5250 2400
-	1    0    0    -1
-$EndComp
 Wire Wire Line
-	5000 2400 5100 2400
+	5000 2400 5150 2400
 Wire Wire Line
-	5400 2400 5500 2400
+	5350 2400 5500 2400
 $Comp
 L Connector:TestPoint TP4
@@
 Wire Notes Line
 	4000 4150 4000 5500
+$Comp
+L Device:Jumper_NC_Small JP1
+U 1 1 5FFB6D8B
+P 5250 2400
+F 0 "JP1" H 5250 2480 50  0000 C CNN
+F 1 "PROG" H 5260 2340 50  0000 C CNN
+F 2 "Jumper:SolderJumper-2_P1.3mm_Bridged_RoundedPad1.0x1.5mm" H 5250 2400 50  0001 C CNN
+F 3 "~" H 5250 2400 50  0001 C CNN
+	1    5250 2400
+	1    0    0    -1
+$EndComp
+Text Notes 4750 2200 0    50   ~ 0
+Cut jumper before programming
 $EndSCHEMATC

Commit message: update touch controller to not use output toggle
Connections:
- net +3V0: no longer U2.6 (TOG)
- no-connect marks 1 -> 2
Other:
- note removed: "PULL TOG HIGH TO TOGGLE OUTPUT\nCURRENT DRAW SEEMS THE SAME FOR BOTH MODES\nEASIER IN CODE TO TOGGLE"
Changed lines of the file:
@@
 	1400 1850 1400 2000
 Connection ~ 1400 2000
-$Comp
-L power:+3V0 #PWR05
-U 1 1 5FE0499E
-P 7000 2700
-F 0 "#PWR05" H 7000 2550 50  0001 C CNN
-F 1 "+3V0" H 7000 2840 50  0000 C CNN
-F 2 "" H 7000 2700 50  0001 C CNN
-F 3 "" H 7000 2700 50  0001 C CNN
-	1    7000 2700
-	1    0    0    -1
-$EndComp
-Wire Wire Line
-	6700 3000 7000 3000
-Wire Wire Line
-	7000 3000 7000 2700
 NoConn ~ 6700 2900
-Text Notes 7000 3500 0    50   ~ 0
-PULL TOG HIGH TO TOGGLE OUTPUT\nCURRENT DRAW SEEMS THE SAME FOR BOTH MODES\nEASIER IN CODE TO TOGGLE
 $Comp
 L Device:C C2
@@
 Wire Wire Line
 	7500 2850 7500 2800
-Wire Notes Line style solid
-	7000 3500 9000 3500
-Wire Notes Line style solid
-	9000 3500 9000 3250
-Wire Notes Line style solid
-	9000 3250 7000 3250
 Text Notes 7500 1850 0    50   ~ 0
 Use C3 to adjust touch sensitivity\n1pF to 50pF suggested in datasheet\n10pF seems to be about right in prototype testing
@@
 Wire Notes Line style solid
 	9450 1850 7500 1850
-Wire Notes Line style solid
-	7000 3050 7000 3500
 Text Notes 8850 2450 0    50   ~ 0
 For touch pad use flood fill on PCB back
@@
 Text Notes 4750 2200 0    50   ~ 0
 Cut jumper before programming
+NoConn ~ 6700 3000
 $EndSCHEMATC

Commit message: pcb layout changes
Parts:
- added JP2, JP4: Jumper_NC_Small, Jumper:SolderJumper-2_P1.3mm_Bridged_RoundedPad1.0x1.5mm, symbol Device:Jumper_NC_Small
- added JP3: Jumper_NC_Small, Jumper:SolderJumper-2_P1.3mm_Open_RoundedPad1.0x1.5mm, symbol Device:Jumper_NO_Small
- added TP6: TestPoint, TestPoint:TestPoint_Pad_3.0x3.0mm, symbol Connector:TestPoint
- J1: footprint TestPoint:TestPoint_THTPad_D2.0mm_Drill1.0mm -> (none)
- JP1: value PROG -> Jumper_NC_Small
Connections:
- net TOUCH: now also JP2.1, JP3.1, JP4.1; no longer C3.1, J1.1
- new net: J1.1, JP4.2
- new net: C3.1, JP2.2
- new net: JP3.2, TP6.1
Other:
- note added: "For touch pad use flood fill"
- note added: "Use C3 to adjust touch sensitivity\n1pF to 50pF suggested in datasheet\nCut JP2 to remove C3 for max sensitivity"
- note added: "optional pad to solder \noffboard tochpad"
- note removed: "For touch pad use flood fill on PCB back"
- note removed: "Use C3 to adjust touch sensitivity\n1pF to 50pF suggested in datasheet\n10pF seems to be about right in prototype testing"
- moved on the sheet: C3
Changed lines of the file:
@@
 F 0 "J1" H 8300 1850 50  0000 C CNN
 F 1 "TOUCH PAD" H 8300 2400 50  0000 C CNN
-F 2 "TestPoint:TestPoint_THTPad_D2.0mm_Drill1.0mm" H 8300 2400 50  0001 C CNN
+F 2 "" H 8300 2400 50  0001 C CNN
 F 3 "" H 8300 2400 50  0001 C CNN
 	1    8300 2400
@@
 $EndComp
 Wire Wire Line
-	6700 2400 7500 2400
+	6700 2400 7150 2400
 Text Label 7000 2400 2    50   ~ 0
 TOUCH
@@
 L Device:C C3
 U 1 1 5FEE0F0C
-P 7500 2650
-F 0 "C3" H 7525 2750 50  0000 L CNN
-F 1 "10p" H 7525 2550 50  0000 L CNN
-F 2 "Capacitor_SMD:C_0603_1608Metric_Pad1.08x0.95mm_HandSolder" H 7538 2500 50  0001 C CNN
-F 3 "~" H 7500 2650 50  0001 C CNN
-	1    7500 2650
-	1    0    0    -1
-$EndComp
-Wire Wire Line
-	7500 2500 7500 2400
-Connection ~ 7500 2400
-Wire Wire Line
-	7500 2400 7700 2400
+P 7150 2900
+F 0 "C3" H 7175 3000 50  0000 L CNN
+F 1 "10p" H 7175 2800 50  0000 L CNN
+F 2 "Capacitor_SMD:C_0603_1608Metric_Pad1.08x0.95mm_HandSolder" H 7188 2750 50  0001 C CNN
+F 3 "~" H 7150 2900 50  0001 C CNN
+	1    7150 2900
+	1    0    0    -1
+$EndComp
+Wire Wire Line
+	7150 2500 7150 2400
 $Comp
 L power:GND #PWR06
 U 1 1 5FEE26DA
-P 7500 2850
-F 0 "#PWR06" H 7500 2600 50  0001 C CNN
-F 1 "GND" H 7500 2700 50  0000 C CNN
-F 2 "" H 7500 2850 50  0001 C CNN
-F 3 "" H 7500 2850 50  0001 C CNN
-	1    7500 2850
-	1    0    0    -1
-$EndComp
-Wire Wire Line
-	7500 2850 7500 2800
-Text Notes 7500 1850 0    50   ~ 0
-Use C3 to adjust touch sensitivity\n1pF to 50pF suggested in datasheet\n10pF seems to be about right in prototype testing
+P 7150 3100
+F 0 "#PWR06" H 7150 2850 50  0001 C CNN
+F 1 "GND" H 7150 2950 50  0000 C CNN
+F 2 "" H 7150 3100 50  0001 C CNN
+F 3 "" H 7150 3100 50  0001 C CNN
+	1    7150 3100
+	1    0    0    -1
+$EndComp
+Wire Wire Line
+	7150 3100 7150 3050
 Wire Notes Line style solid
-	7500 2350 7500 1600
+	8950 3050 8950 3300
 Wire Notes Line style solid
-	7500 1600 9450 1600
-Wire Notes Line style solid
-	9450 1600 9450 1850
-Wire Notes Line style solid
-	9450 1850 7500 1850
+	8950 3300 7300 3300
 Text Notes 8850 2450 0    50   ~ 0
-For touch pad use flood fill on PCB back
+For touch pad use flood fill
 Wire Wire Line
 	5000 2400 5150 2400
@@
 P 5250 2400
 F 0 "JP1" H 5250 2480 50  0000 C CNN
-F 1 "PROG" H 5260 2340 50  0000 C CNN
+F 1 "Jumper_NC_Small" H 5260 2340 50  0001 C CNN
 F 2 "Jumper:SolderJumper-2_P1.3mm_Bridged_RoundedPad1.0x1.5mm" H 5250 2400 50  0001 C CNN
 F 3 "~" H 5250 2400 50  0001 C CNN
@@
 Cut jumper before programming
 NoConn ~ 6700 3000
+Wire Notes Line style solid
+	7300 3300 7300 3050
+Wire Notes Line style solid
+	7300 3050 8950 3050
+Text Notes 7300 3300 0    50   ~ 0
+Use C3 to adjust touch sensitivity\n1pF to 50pF suggested in datasheet\nCut JP2 to remove C3 for max sensitivity
+Wire Wire Line
+	7150 2750 7150 2700
+$Comp
+L Device:Jumper_NC_Small JP2
+U 1 1 5FF05A9A
+P 7150 2600
+F 0 "JP2" H 7150 2680 50  0000 C CNN
+F 1 "Jumper_NC_Small" H 7160 2540 50  0001 C CNN
+F 2 "Jumper:SolderJumper-2_P1.3mm_Bridged_RoundedPad1.0x1.5mm" H 7150 2600 50  0001 C CNN
+F 3 "~" H 7150 2600 50  0001 C CNN
+	1    7150 2600
+	0    1    1    0
+$EndComp
+$Comp
+L Device:Jumper_NC_Small JP4
+U 1 1 5FF37EA2
+P 7550 2400
+F 0 "JP4" H 7550 2480 50  0000 C CNN
+F 1 "Jumper_NC_Small" H 7560 2340 50  0001 C CNN
+F 2 "Jumper:SolderJumper-2_P1.3mm_Bridged_RoundedPad1.0x1.5mm" H 7550 2400 50  0001 C CNN
+F 3 "~" H 7550 2400 50  0001 C CNN
+	1    7550 2400
+	1    0    0    -1
+$EndComp
+$Comp
+L Device:Jumper_NO_Small JP3
+U 1 1 5FF38261
+P 7150 2250
+F 0 "JP3" H 7150 2330 50  0000 C CNN
+F 1 "Jumper_NC_Small" H 7160 2190 50  0001 C CNN
+F 2 "Jumper:SolderJumper-2_P1.3mm_Open_RoundedPad1.0x1.5mm" H 7150 2250 50  0001 C CNN
+F 3 "~" H 7150 2250 50  0001 C CNN
+	1    7150 2250
+	0    -1   -1   0
+$EndComp
+Connection ~ 7150 2400
+Wire Wire Line
+	7650 2400 7700 2400
+Wire Wire Line
+	7150 2350 7150 2400
+Text Notes 7000 1750 0    50   ~ 0
+optional pad to solder \noffboard tochpad
+Wire Wire Line
+	7150 2400 7450 2400
+$Comp
+L Connector:TestPoint TP6
+U 1 1 5FF5D320
+P 7150 2100
+F 0 "TP6" H 7150 2370 50  0000 C CNN
+F 1 "TestPoint" H 7150 2300 50  0000 C CNN
+F 2 "TestPoint:TestPoint_Pad_3.0x3.0mm" H 7350 2100 50  0001 C CNN
+F 3 "~" H 7350 2100 50  0001 C CNN
+	1    7150 2100
+	1    0    0    -1
+$EndComp
+Wire Wire Line
+	7150 2100 7150 2150
 $EndSCHEMATC
